Commit message: Remove all the collision from iCubGazeboV2_5 model

File: iCub/robots/iCubGazeboV2_5/model.urdf (robot description, URDF)
Before this commit: robot iCub, 189 links, 188 joints
Links:
- link chest: geometry visual mesh filename=package://iCub/meshes/simmechanics/sim_sea_2-5_chest_bb_prt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 scale=0.001 0.001 0.001
- link head: geometry visual mesh filename=package://iCub/meshes/simmechanics/sim_sea_2-5_head_prt-bin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 scale=0.001 0.001 0.001
- link l_ankle_1: geometry visual mesh filename=package://iCub/meshes/simmechanics/sim_sea_2-5_l_ankle_prt-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 scale=0.001 0.001 0.001
- link l_ankle_2: geometry visual mesh filename=package://iCub/meshes/simmechanics/sim_sea_2-5_l_foot_prt-b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 scale=0.001 0.001 0.001
- link l_elbow_1: geometry visual mesh filename=package://iCub/meshes/simmechanics/sim_sea_2-5_l_elbow_pros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 scale=0.001 0.001 0.001
- link l_forearm: geometry visual mesh filename=package://iCub/meshes/simmechanics/sim_sea_2-5_l_forearm_pr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 scale=0.001 0.001 0.001
- link l_hand: geometry visual mesh filename=package://iCub/meshes/simmechanics/sim_sea_2-5_l_hand_prt-b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 scale=0.001 0.001 0.001
- link l_hip_1: geometry visual mesh filename=package://iCub/meshes/simmechanics/sim_sea_2-5_l_hip_1_prt-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 scale=0.001 0.001 0.001
- link l_hip_2: geometry visual mesh filename=package://iCub/meshes/simmechanics/sim_sea_2-5_l_hip_2_prt-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 scale=0.001 0.001 0.001
- link l_hip_3: geometry visual mesh filename=package://iCub/meshes/simmechanics/sim_sea_2-5_l_upper_thig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 scale=0.001 0.001 0.001
- link l_lower_leg: geometry visual mesh filename=package://iCub/meshes/simmechanics/sim_sea_2-5_l_shank_prt-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 scale=0.001 0.001 0.001
- link l_shoulder_1: geometry visual mesh filename=package://iCub/meshes/simmechanics/sim_sea_2-5_l_shoulder_1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 scale=0.001 0.001 0.001
- link l_shoulder_2: geometry visual mesh filename=package://iCub/meshes/simmechanics/sim_sea_2-5_l_shoulder_2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 scale=0.001 0.001 0.001
- link l_shoulder_3: geometry visual mesh filename=package://iCub/meshes/simmechanics/sim_sea_2-5_l_upper_arm_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 scale=0.001 0.001 0.001
- link l_upper_arm: geometry visual mesh filename=package://iCub/meshes/simmechanics/sim_sea_2-5_l_elbow_prt-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 scale=0.001 0.001 0.001
- link l_upper_leg: geometry visual mesh filename=package://iCub/meshes/simmechanics/sim_sea_2-5_l_thigh_prt-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 scale=0.001 0.001 0.001
- link l_wrist_1: geometry visual mesh filename=package://iCub/meshes/simmechanics/sim_sea_2-5_l_wrist_pitc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 scale=0.001 0.001 0.001
- link neck_1: geometry visual mesh filename=package://iCub/meshes/simmechanics/sim_sea_2-5_neck_1_prt-b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 scale=0.001 0.001 0.001
- link neck_2: geometry visual mesh filename=package://iCub/meshes/simmechanics/sim_sea_2-5_neck_2_prt-b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 scale=0.001 0.001 0.001
- link r_ankle_1: geometry visual mesh filename=package://iCub/meshes/simmechanics/sim_sea_2-5_r_ankle_prt-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 scale=0.001 0.001 0.001
- link r_ankle_2: geometry visual mesh filename=package://iCub/meshes/simmechanics/sim_sea_2-5_r_foot_prt-b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 scale=0.001 0.001 0.001
- link r_elbow_1: geometry visual mesh filename=package://iCub/meshes/simmechanics/sim_sea_2-5_r_elbow_pros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 scale=0.001 0.001 0.001
- link r_forearm: geometry visual mesh filename=package://iCub/meshes/simmechanics/sim_sea_2-5_r_forearm_pr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 scale=0.001 0.001 0.001
- link r_hand: geometry visual mesh filename=package://iCub/meshes/simmechanics/sim_sea_2-5_r_hand_prt-b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 scale=0.001 0.001 0.001
- link r_hip_1: geometry visual mesh filename=package://iCub/meshes/simmechanics/sim_sea_2-5_r_hip_1_prt-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 scale=0.001 0.001 0.001
- link r_hip_2: geometry visual mesh filename=package://iCub/meshes/simmechanics/sim_sea_2-5_r_hip_2_prt-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 scale=0.001 0.001 0.001
- link r_hip_3: geometry visual mesh filename=package://iCub/meshes/simmechanics/sim_sea_2-5_r_upper_thig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 scale=0.001 0.001 0.001
- link r_lower_leg: geometry visual mesh filename=package://iCub/meshes/simmechanics/sim_sea_2-5_r_shank_prt-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 scale=0.001 0.001 0.001
- link r_shoulder_1: geometry visual mesh filename=package://iCub/meshes/simmechanics/sim_sea_2-5_r_shoulder_1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 scale=0.001 0.001 0.001
- link r_shoulder_2: geometry visual mesh filename=package://iCub/meshes/simmechanics/sim_sea_2-5_r_shoulder_2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 scale=0.001 0.001 0.001
- link r_shoulder_3: geometry visual mesh filename=package://iCub/meshes/simmechanics/sim_sea_2-5_r_upper_arm_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 scale=0.001 0.001 0.001
- link r_upper_arm: geometry visual mesh filename=package://iCub/meshes/simmechanics/sim_sea_2-5_r_elbow_prt-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 scale=0.001 0.001 0.001
- link r_upper_leg: geometry visual mesh filename=package://iCub/meshes/simmechanics/sim_sea_2-5_r_thigh_prt-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 scale=0.001 0.001 0.001
- link r_wrist_1: geometry visual mesh filename=package://iCub/meshes/simmechanics/sim_sea_2-5_r_wrist_pitc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 scale=0.001 0.001 0.001
- link root_link: geometry visual mesh filename=package://iCub/meshes/simmechanics/sim_sea_2-5_root_link_pr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 scale=0.001 0.001 0.001
- link torso_1: geometry visual mesh filename=package://iCub/meshes/simmechanics/sim_sea_2-5_lap_belt_1_p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 scale=0.001 0.001 0.001
- link torso_2: geometry visual mesh filename=package://iCub/meshes/simmechanics/sim_sea_2-5_lap_belt_2_p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 scale=0.001 0.001 0.001

Commit message: Update the kp coefficent and add a frame in the center of the contact surface

File: iCub/robots/iCubGazeboV2_5/model.urdf (robot description, URDF)
Before this commit: robot iCub, 189 links, 188 joints
Links:
- added link l_sole_ground_middle
- added link r_sole_ground_middle
Joints:
- added joint l_sole_ground_middle_fixed_joint: type fixed, parent l_foot, child l_sole_ground_middle, origin xyz=0.03 -0.005 0.014 rpy=-3.14159265359 0 0
- added joint r_sole_ground_middle_fixed_joint: type fixed, parent r_foot, child r_sole_ground_middle, origin xyz=0.03 0.005 0.014 rpy=-3.14159265359 0 0
