Commit message: add temporarily head IMU for iCubGazeboV3

File: iCub/robots/iCubGazeboV3/model.urdf (robot description, URDF)
Before this commit: robot iCub, 45 links, 44 joints
Links:
- added link imu_frame
Joints:
- added joint imu_frame_fixed_joint: type fixed, parent head, child imu_frame, origin xyz=0.009500000190735 0.133444 0.009299999999999996 rpy=-1.5707963267948961 1.570796326794896 0
